Commit message: updates

File: urdf/inertia.xacro (robot description, xacro)
@@ -14,7 +14,34 @@
     </inertial>
   </xacro:macro>
+  <xacro:macro name="sphere_inertial_roll" params="mass radius roll">
+    <inertial>
+      <origin xyz="0 0 0" rpy="${roll} 0 0"/> <mass value="${mass}"/>
+      <inertia
+        ixx="${(2/5) * mass * (radius*radius)}"
+        ixy="0.0"
+        ixz="0.0"
+        iyy="${(2/5) * mass * (radius*radius)}"
+        iyz="0.0"
+        izz="${(2/5) * mass * (radius*radius)}"
+      />
+    </inertial>
+  </xacro:macro>
   <xacro:macro name="cylinder_inertial" params="mass radius length">
     <inertial>
       <origin xyz="0 0 0" rpy="0 0 0"/>
+      <mass value="${mass}"/>
+      <inertia
+        ixx="${(1/12) * mass * (3*radius*radius + length*length)}"
+        ixy="0.0"
+        ixz="0.0"
+        iyy="${(1/12) * mass * (3*radius*radius + length*length)}"
+        iyz="0.0"
+        izz="${(1/2) * mass * (radius*radius)}"
+      />
+    </inertial>
+  </xacro:macro>
+  <xacro:macro name="cylinder_inertial_roll" params="mass radius length roll">
+    <inertial>
+      <origin xyz="0 0 0" rpy="${roll} 0 0"/>
       <mass value="${mass}"/>
       <inertia

File: urdf/marrtino.urdf.xacro (robot description, xacro)
@@ -34,5 +34,22 @@
         <origin xyz="0.0 0.0 0.0" rpy="0.0 0.0 0.0"/>
     </collision>
-    <xacro:box_inertial mass="0.5" x_dim="${base_l}" y_dim="${base_w}" z_dim="${base_h}"/>
+    <xacro:box_inertial mass="0.2" x_dim="${base_l}" y_dim="${base_w}" z_dim="${base_h}"/>
+  </link>
+  <!-- to balance weight on the bottom and between the wheels -->
+  <link name="battery_link">
+    <visual>
+        <geometry>
+            <box size="${base_l/4} ${base_w/4} ${base_h/4}"/>
+        </geometry>
+        <origin xyz="0.0 0.0 0.0" rpy="0.0 0.0 0.0"/>
+        <material name="black"/>
+    </visual>
+    <collision>
+        <geometry>
+            <box size="${base_l/4} ${base_w/4} ${base_h/4}"/>
+        </geometry>
+        <origin xyz="0.0 0.0 0.0" rpy="0.0 0.0 0.0"/>
+    </collision>
+    <xacro:box_inertial mass="0.3" x_dim="${base_l/4}" y_dim="${base_w/4}" z_dim="${base_h/4}"/>
   </link>
   <link name="left_wheel">
@@ -107,4 +124,9 @@
     <origin xyz="0.0 0.0 ${base_h/2+wheel_r}" rpy="0.0 0.0 0.0"/>
   </joint>
+  <joint name="battery_joint" type="fixed">
+    <parent link="base_footprint"/>
+    <child link="battery_link"/>
+    <origin xyz="${base_l/4} 0.0 ${wheel_r*2}" rpy="0.0 0.0 0.0"/>
+  </joint>
   <joint name="left_wheel_joint" type="continuous">
     <parent link="base_link"/>
