Commit message: position, velocity control

File: marrtino_gazebo/urdf/marrtino_2_arms.urdf.xacro (robot description, xacro)
@@ -3,4 +3,10 @@
   <xacro:arg name="namespace" default="" />
   <xacro:include filename="$(find marrtino_gazebo)/urdf/marrtino_base.urdf.xacro" />
+  <xacro:property name="wheel_r" value="0.06" />
+  <xacro:property name="wheel_max_velocity" value="${1 / wheel_r}" /> <!-- 1/r rad/s -> 1 m/s -->
+  <xacro:property name="arm_lower_limit" value="${-5*pi/4}" />
+  <xacro:property name="arm_upper_limit" value="${pi/4}" />
+  <xacro:property name="arm_max_effort" value="100" />
+  <xacro:property name="arm_max_velocity" value="1.0" />
   <xacro:marrtino_base />
   <xacro:marrtino_sensors />
@@ -15,6 +21,4 @@
     </plugin>
   </gazebo>
-  <xacro:property name="max_wheel_velocity" value="10.0" />
-  <xacro:property name="max_arm_effort" value="100.0" />
   <ros2_control name="GazeboSimSystem" type="system">
     <hardware>
@@ -23,6 +27,6 @@
     <joint name="left_wheel_joint">
       <command_interface name="velocity">
-        <param name="min">${-max_wheel_velocity}</param>
-        <param name="max">${max_wheel_velocity}</param>
+        <param name="min">${-wheel_max_velocity}</param>
+        <param name="max">${wheel_max_velocity}</param>
       </command_interface>
       <state_interface name="position"/>
@@ -31,6 +35,6 @@
     <joint name="right_wheel_joint">
       <command_interface name="velocity">
-        <param name="min">${-max_wheel_velocity}</param>
-        <param name="max">${max_wheel_velocity}</param>
+        <param name="min">${-wheel_max_velocity}</param>
+        <param name="max">${wheel_max_velocity}</param>
       </command_interface>
       <state_interface name="position"/>
@@ -39,10 +43,14 @@
     <joint name="left_arm_joint">
       <command_interface name="effort">
-        <param name="min">${-max_arm_effort}</param>
-        <param name="max">${max_arm_effort}</param>
+        <param name="min">${-arm_max_effort}</param>
+        <param name="max">${arm_max_effort}</param>
+      </command_interface>
+      <command_interface name="velocity">
+        <param name="min">${-arm_max_velocity}</param>
+        <param name="max">${arm_max_velocity}</param>
       </command_interface>
       <command_interface name="position">
-        <param name="min">${-pi}</param>
-        <param name="max">${pi}</param>
+        <param name="min">${arm_lower_limit}</param>
+        <param name="max">${arm_upper_limit}</param>
       </command_interface>
       <state_interface name="position"/>
@@ -51,10 +59,14 @@
     <joint name="right_arm_joint">
       <command_interface name="effort">
-        <param name="min">${-max_arm_effort}</param>
-        <param name="max">${max_arm_effort}</param>
+        <param name="min">${-arm_max_effort}</param>
+        <param name="max">${arm_max_effort}</param>
+      </command_interface>
+      <command_interface name="velocity">
+        <param name="min">${-arm_max_velocity}</param>
+        <param name="max">${arm_max_velocity}</param>
       </command_interface>
       <command_interface name="position">
-        <param name="min">${-pi}</param>
-        <param name="max">${pi}</param>
+        <param name="min">${arm_lower_limit}</param>
+        <param name="max">${arm_upper_limit}</param>
       </command_interface>
       <state_interface name="position"/>

File: marrtino_gazebo/urdf/marrtino_base.urdf.xacro (robot description, xacro)
@@ -14,10 +14,8 @@
   <xacro:property name="base_h" value="0.20" />
   <xacro:macro name="marrtino_base">
-      <xacro:property name="wheel_r" value="0.06" />
       <xacro:property name="wheel_l" value="0.03" />
-      <xacro:property name="friction" value="0.01" />
-      <xacro:property name="damping" value="0.05" />
-      <xacro:property name="max_effort" value="1000.0" />
-      <xacro:property name="max_velocity" value="10.0" />
+      <xacro:property name="wheel_friction" value="0.01" />
+      <xacro:property name="wheel_damping" value="0.05" />
+      <xacro:property name="wheel_max_effort" value="100.0" />
       <link name="base_footprint"/>
       <link name="base_link">
@@ -117,6 +115,6 @@
         <origin xyz="${base_l/4} ${base_w/2+wheel_l/2} ${-base_h/2}" rpy="0 0.0 0.0"/>
         <axis xyz="0.0 1.0 0.0"/>
-        <dynamics damping="${damping}" friction="${friction}"/>
-        <limit effort="${max_effort}" velocity="${max_velocity}"/>
+        <dynamics damping="${wheel_damping}" friction="${wheel_friction}"/>
+        <limit effort="${wheel_max_effort}" velocity="${wheel_max_velocity}"/>
       </joint>
       <joint name="right_wheel_joint" type="continuous">
@@ -125,6 +123,6 @@
         <origin xyz="${base_l/4} ${-base_w/2-wheel_l/2} ${-base_h/2}" rpy="0 0.0 0.0"/>
         <axis xyz="0.0 1.0 0.0"/>
-        <dynamics damping="${damping}" friction="${friction}"/>
-        <limit effort="${max_effort}" velocity="${max_velocity}"/>
+        <dynamics damping="${wheel_damping}" friction="${wheel_friction}"/>
+        <limit effort="${wheel_max_effort}" velocity="${wheel_max_velocity}"/>
       </joint>
       <joint name="caster_wheel_joint" type="fixed">
@@ -168,4 +166,6 @@
       <xacro:property name="arm_length" value="0.2" />
       <xacro:property name="arm_mass" value="0.05" />
+      <xacro:property name="arm_friction" value="0.01" />
+      <xacro:property name="arm_damping" value="0.02" />
       <link name="left_arm_body">
         <visual>
@@ -253,7 +253,7 @@
         <origin xyz="0.1 ${0.221+arm_radius} 0.07" rpy="0 0 0"/>
         <axis xyz="0.0 1.0 0.0"/>
-        <dynamics damping="0.02" friction="0.01"/>
-        <limit lower="${-5*pi/4}" upper="${pi/4}"
-            effort="100" velocity="1.0"/>
+        <dynamics friction="${arm_friction}" damping="${arm_damping}" />
+        <limit lower="${arm_lower_limit}" upper="${arm_upper_limit}"
+            effort="${arm_max_effort}" velocity="${arm_max_velocity}"/>
       </joint>
       <joint name="left_arm_body_joint" type="fixed">
@@ -272,7 +272,7 @@
         <origin xyz="0.1 ${-(0.221+arm_radius)} 0.07" rpy="0 0 0"/>
         <axis xyz="0.0 1.0 0.0"/>
-        <dynamics damping="0.02" friction="0.01"/>
-        <limit lower="${-5*pi/4}" upper="${pi/4}"
-            effort="100" velocity="1.0"/>
+        <dynamics friction="${arm_friction}" damping="${arm_damping}" />
+        <limit lower="${arm_lower_limit}" upper="${arm_upper_limit}"
+            effort="${arm_max_effort}" velocity="${arm_max_velocity}"/>
       </joint>
       <joint name="right_arm_body_joint" type="fixed">

File: marrtino_gazebo/urdf/smarrtino.urdf.xacro (robot description, xacro)
@@ -9,8 +9,8 @@
   <xacro:property name="wheel_r" value="0.05" />
   <xacro:property name="wheel_l" value="0.02" />
-  <xacro:property name="friction" value="0.001" />
-  <xacro:property name="damping" value="0.001" />
-  <xacro:property name="max_effort" value="1000.0" />
-  <xacro:property name="max_velocity" value="10.0" />
+  <xacro:property name="wheel_friction" value="0.001" />
+  <xacro:property name="wheel_damping" value="0.001" />
+  <xacro:property name="wheel_max_effort" value="100.0" />
+  <xacro:property name="wheel_max_velocity" value="${1 / wheel_r}" /> <!-- 1/r rad/s -> 1 m/s -->
   <xacro:property name="arm_mass" value="0.08" />
   <xacro:property name="arm_radius" value="0.02" />
@@ -20,4 +20,6 @@
   <xacro:property name="arm_friction" value="0.001" />
   <xacro:property name="arm_damping" value="0.01" />
+  <xacro:property name="arm_lower_limit" value="${-5*pi/4}" />
+  <xacro:property name="arm_upper_limit" value="${pi/4}" />
   <xacro:property name="head_mass" value="0.10" />
   <xacro:property name="head_radius" value="0.05" />
@@ -26,4 +28,8 @@
   <xacro:property name="head_friction" value="0.02" />
   <xacro:property name="head_damping" value="0.02" />
+  <xacro:property name="head_pan_lower_limit" value="${-pi/2}" />
+  <xacro:property name="head_pan_upper_limit" value="${pi/2}" />
+  <xacro:property name="head_tilt_lower_limit" value="${-pi/4}" />
+  <xacro:property name="head_tilt_upper_limit" value="${pi/4}" />
   <xacro:include filename="$(find marrtino_gazebo)/urdf/inertia.xacro" />
   <material name="orange"><color rgba="1.0 0.33 0.0 1.0"/></material>
@@ -202,5 +208,5 @@
     <dynamics damping="${head_damping}" friction="${head_friction}"/>
     <limit effort="${head_max_effort}" velocity="${head_max_velocity}"
-           lower="${-pi/4}" upper="${pi/4}" />
+           lower="${head_tilt_lower_limit}" upper="${head_tilt_upper_limit}" />
   </joint>
   <joint name="pan_head_joint" type="revolute">
@@ -211,5 +217,5 @@
     <dynamics damping="${head_damping}" friction="${head_friction}"/>
     <limit effort="${head_max_effort}" velocity="${head_max_velocity}"
-           lower="${-pi/2}" upper="${pi/2}" />
+           lower="${head_pan_lower_limit}" upper="${head_pan_upper_limit}" />
   </joint>
   <joint name="base_head_joint" type="fixed">
@@ -223,6 +229,6 @@
     <origin xyz="0 ${base_w/2+wheel_l/2} ${wheel_r}" rpy="0 0.0 0.0"/>
     <axis xyz="0.0 1.0 0.0"/>
-    <dynamics damping="${damping}" friction="${friction}"/>
-    <limit effort="${max_effort}" velocity="${max_velocity}"/>
+    <dynamics damping="${wheel_damping}" friction="${wheel_friction}"/>
+    <limit effort="${wheel_max_effort}" velocity="${wheel_max_velocity}"/>
   </joint>
   <joint name="right_wheel_joint" type="continuous">
@@ -231,6 +237,6 @@
     <origin xyz="0 ${-base_w/2-wheel_l/2} ${wheel_r}" rpy="0 0.0 0.0"/>
     <axis xyz="0.0 1.0 0.0"/>
-    <dynamics damping="${damping}" friction="${friction}"/>
-    <limit effort="${max_effort}" velocity="${max_velocity}"/>
+    <dynamics damping="${wheel_damping}" friction="${wheel_friction}"/>
+    <limit effort="${wheel_max_effort}" velocity="${wheel_max_velocity}"/>
   </joint>
   <joint name="caster_wheel_joint" type="fixed">
@@ -340,5 +346,5 @@
     <dynamics damping="${arm_damping}" friction="${arm_friction}"/>
     <limit effort="${arm_max_effort}" velocity="${arm_max_velocity}"
-           lower="${-5*pi/4}" upper="${pi/4}" />
+           lower="${arm_lower_limit}" upper="${arm_upper_limit}" />
   </joint>
   <joint name="right_arm_joint" type="revolute">
@@ -349,5 +355,5 @@
     <dynamics damping="${arm_damping}" friction="${arm_friction}"/>
     <limit effort="${arm_max_effort}" velocity="${arm_max_velocity}"
-           lower="${-5*pi/4}" upper="${pi/4}" />
+           lower="${arm_lower_limit}" upper="${arm_upper_limit}" />
   </joint>
   <joint name="left_arm_body_joint" type="fixed">
@@ -367,6 +373,6 @@
     <joint name="left_wheel_joint">
       <command_interface name="velocity">
-        <param name="min">${-max_velocity}</param>
-        <param name="max">${max_velocity}</param>
+        <param name="min">${-wheel_max_velocity}</param>
+        <param name="max">${wheel_max_velocity}</param>
       </command_interface>
       <state_interface name="position"/>
@@ -375,6 +381,6 @@
     <joint name="right_wheel_joint">
       <command_interface name="velocity">
-        <param name="min">${-max_velocity}</param>
-        <param name="max">${max_velocity}</param>
+        <param name="min">${-wheel_max_velocity}</param>
+        <param name="max">${wheel_max_velocity}</param>
       </command_interface>
       <state_interface name="position"/>
@@ -383,6 +389,14 @@
     <joint name="left_arm_joint">
       <command_interface name="effort">
-        <param name="min">-10</param>
-        <param name="max">10</param>
+        <param name="min">${-arm_max_effort}</param>
+        <param name="max">${arm_max_effort}</param>
+      </command_interface>
+      <command_interface name="velocity">
+        <param name="min">${-arm_max_velocity}</param>
+        <param name="max">${arm_max_velocity}</param>
+      </command_interface>
+      <command_interface name="position">
+        <param name="min">${arm_lower_limit}</param>
+        <param name="max">${arm_upper_limit}</param>
       </command_interface>
       <state_interface name="position"/>
@@ -391,6 +405,14 @@
     <joint name="right_arm_joint">
       <command_interface name="effort">
-        <param name="min">-10</param>
-        <param name="max">10</param>
+        <param name="min">${-arm_max_effort}</param>
+        <param name="max">${arm_max_effort}</param>
+      </command_interface>
+      <command_interface name="velocity">
+        <param name="min">${-arm_max_velocity}</param>
+        <param name="max">${arm_max_velocity}</param>
+      </command_interface>
+      <command_interface name="position">
+        <param name="min">${arm_lower_limit}</param>
+        <param name="max">${arm_upper_limit}</param>
       </command_interface>
       <state_interface name="position"/>
@@ -399,6 +421,14 @@
     <joint name="pan_head_joint">
       <command_interface name="effort">
-        <param name="min">-10</param>
-        <param name="max">10</param>
+        <param name="min">${-head_max_effort}</param>
+        <param name="max">${head_max_effort}</param>
+      </command_interface>
+      <command_interface name="velocity">
+        <param name="min">${-head_max_velocity}</param>
+        <param name="max">${head_max_velocity}</param>
+      </command_interface>
+      <command_interface name="position">
+        <param name="min">${head_pan_lower_limit}</param>
+        <param name="max">${head_pan_upper_limit}</param>
       </command_interface>
       <state_interface name="position"/>
@@ -407,6 +437,14 @@
     <joint name="tilt_head_joint">
       <command_interface name="effort">
-        <param name="min">-10</param>
-        <param name="max">10</param>
+        <param name="min">${-head_max_effort}</param>
+        <param name="max">${head_max_effort}</param>
+      </command_interface>
+      <command_interface name="velocity">
+        <param name="min">${-head_max_velocity}</param>
+        <param name="max">${head_max_velocity}</param>
+      </command_interface>
+      <command_interface name="position">
+        <param name="min">${head_tilt_lower_limit}</param>
+        <param name="max">${head_tilt_upper_limit}</param>
       </command_interface>
       <state_interface name="position"/>
