Commit message: params

File: marrtino_gazebo/urdf/marrtino.urdf.xacro (robot description, xacro)
@@ -166,6 +166,6 @@
     <joint name="left_wheel_joint">
       <command_interface name="velocity">
-        <param name="min">-1</param>
-        <param name="max">1</param>
+        <param name="min">${-max_velocity}</param>
+        <param name="max">${max_velocity}</param>
       </command_interface>
       <state_interface name="position"/>
@@ -174,6 +174,6 @@
     <joint name="right_wheel_joint">
       <command_interface name="velocity">
-        <param name="min">-1</param>
-        <param name="max">1</param>
+        <param name="min">${-max_velocity}</param>
+        <param name="max">${max_velocity}</param>
       </command_interface>
       <state_interface name="position"/>

File: marrtino_gazebo/urdf/smarrtino.urdf.xacro (robot description, xacro)
@@ -12,5 +12,5 @@
   <xacro:property name="damping" value="0.001" />
   <xacro:property name="max_effort" value="1000.0" />
-  <xacro:property name="max_velocity" value="100.0" />
+  <xacro:property name="max_velocity" value="10.0" />
   <xacro:property name="arm_mass" value="0.08" />
   <xacro:property name="arm_radius" value="0.02" />

Commit message: marrtino 2 arms

File: marrtino_gazebo/urdf/marrtino.urdf.xacro (robot description, xacro)
@@ -2,162 +2,16 @@
 <robot name="marrtino" xmlns:xacro="http://ros.org/wiki/xacro">
   <xacro:arg name="namespace" default="" />
-  <xacro:property name="base_w" value="0.40" />
-  <xacro:property name="base_l" value="0.30" />
-  <xacro:property name="base_h" value="0.20" />
-  <xacro:property name="wheel_r" value="0.06" />
-  <xacro:property name="wheel_l" value="0.03" />
-  <xacro:property name="friction" value="0.01" />
-  <xacro:property name="damping" value="0.05" />
-  <xacro:property name="max_effort" value="1000.0" />
-  <xacro:property name="max_velocity" value="10.0" />
-  <xacro:include filename="$(find marrtino_gazebo)/urdf/inertia.xacro" />
-  <material name="orange"><color rgba="1.0 0.33 0.0 1.0"/></material>
-  <material name="red"><color rgba="0.8 0 0 1"/></material>
-  <material name="green"><color rgba="0 1 0 1"/></material>
-  <material name="blue"><color rgba="0 0 1 1"/></material>
-  <material name="black"><color rgba="0 0 0 1.0"/></material>
-  <material name="grey"><color rgba="0.7 0.7 0.7 1.0"/></material>
-  <material name="white"><color rgba="1 1 1 1.0"/></material>
-  <link name="base_footprint"/>
-  <link name="base_link">
-    <visual>
-        <geometry>
-            <box size="${base_l} ${base_w} ${base_h}"/>
-        </geometry>
-        <origin xyz="0.0 0.0 0.0" rpy="0.0 0.0 0.0"/>
-        <material name="red"/>
-    </visual>
-    <collision>
-        <geometry>
-            <box size="${base_l} ${base_w} ${base_h}"/>
-        </geometry>
-        <origin xyz="0.0 0.0 0.0" rpy="0.0 0.0 0.0"/>
-    </collision>
-    <xacro:box_inertial mass="0.2" x_dim="${base_l}" y_dim="${base_w}" z_dim="${base_h}"/>
-  </link>
-  <!-- to balance weight on the bottom and between the wheels -->
-  <link name="battery_link">
-    <visual>
-        <geometry>
-            <box size="${base_l/4} ${base_w/4} ${base_h/4}"/>
-        </geometry>
-        <origin xyz="0.0 0.0 0.0" rpy="0.0 0.0 0.0"/>
-        <material name="black"/>
-    </visual>
-    <collision>
-        <geometry>
-            <box size="${base_l/4} ${base_w/4} ${base_h/4}"/>
-        </geometry>
-        <origin xyz="0.0 0.0 0.0" rpy="0.0 0.0 0.0"/>
-    </collision>
-    <xacro:box_inertial mass="0.3" x_dim="${base_l/4}" y_dim="${base_w/4}" z_dim="${base_h/4}"/>
-  </link>
-  <link name="left_wheel">
-    <visual>
-        <geometry>
-            <cylinder radius="${wheel_r}" length="${wheel_l}"/>
-        </geometry>
-        <origin xyz="0.0 0.0 0.0" rpy="1.57 0.0 0.0"/>
-        <material name="black"/>
-    </visual>
-    <collision>
-        <geometry>
-            <cylinder radius="${wheel_r}" length="${wheel_l}"/>
-        </geometry>
-        <origin xyz="0.0 0.0 0.0" rpy="1.57 0.0 0.0"/>
-    </collision>
-    <xacro:cylinder_inertial mass="0.3" radius="${wheel_r}" length="${wheel_l}"/>
-  </link>
-  <link name="right_wheel">
-    <visual>
-        <geometry>
-            <cylinder radius="${wheel_r}" length="${wheel_l}"/>
-        </geometry>
-        <origin xyz="0.0 0.0 0.0" rpy="1.57 0.0 0.0"/>
-        <material name="black"/>
-    </visual>
-    <collision>
-        <geometry>
-            <cylinder radius="${wheel_r}" length="${wheel_l}"/>
-        </geometry>
-        <origin xyz="0.0 0.0 0.0" rpy="1.57 0.0 0.0"/>
-    </collision>
-    <xacro:cylinder_inertial mass="0.3" radius="${wheel_r}" length="${wheel_l}"/>
-  </link>
-  <link name="caster_wheel">
-    <visual>
-        <geometry>
-            <sphere radius="${wheel_r/2}"/>
-        </geometry>
-        <origin xyz="0.0 0.0 0.0" rpy="0.0 0.0 0.0"/>
-        <material name="black"/>
-    </visual>
-    <collision>
-        <geometry>
-            <sphere radius="${wheel_r/2}"/>
-        </geometry>
-        <origin xyz="0.0 0.0 0.0" rpy="0.0 0.0 0.0"/>
-    </collision>
-    <xacro:sphere_inertial mass="0.1" radius="${wheel_r/2}" />
-  </link>
-  <link name="imu_link">
-    <visual>
-      <origin rpy="0 0 0" xyz="0 0 0.0"/>
-      <geometry>
-        <box size="0.04 0.04 0.02"/>
-      </geometry>
-      <material name="green"/>
-    </visual>
-  </link>
-  <link name="lidar_link">
-    <visual>
-        <geometry>
-            <cylinder radius="0.05" length="0.04"/>
-        </geometry>
-        <origin xyz="0.0 0.0 0.0" rpy="0.0 0.0 0.0"/>
-        <material name="white"/>
-    </visual>
-  </link>
-  <joint name="base_joint" type="fixed">
-    <parent link="base_footprint"/>
-    <child link="base_link"/>
-    <origin xyz="0.0 0.0 ${base_h/2+wheel_r}" rpy="0.0 0.0 0.0"/>
-  </joint>
-  <joint name="battery_joint" type="fixed">
-    <parent link="base_footprint"/>
-    <child link="battery_link"/>
-    <origin xyz="${base_l/4} 0.0 ${wheel_r*2}" rpy="0.0 0.0 0.0"/>
-  </joint>
-  <joint name="left_wheel_joint" type="continuous">
-    <parent link="base_link"/>
-    <child link="left_wheel"/>
-    <origin xyz="${base_l/4} ${base_w/2+wheel_l/2} ${-base_h/2}" rpy="0 0.0 0.0"/>
-    <axis xyz="0.0 1.0 0.0"/>
-    <dynamics damping="${damping}" friction="${friction}"/>
-    <limit effort="${max_effort}" velocity="${max_velocity}"/>
-  </joint>
-  <joint name="right_wheel_joint" type="continuous">
-    <parent link="base_link"/>
-    <child link="right_wheel"/>
-    <origin xyz="${base_l/4} ${-base_w/2-wheel_l/2} ${-base_h/2}" rpy="0 0.0 0.0"/>
-    <axis xyz="0.0 1.0 0.0"/>
-    <dynamics damping="${damping}" friction="${friction}"/>
-    <limit effort="${max_effort}" velocity="${max_velocity}"/>
-  </joint>
-  <joint name="caster_wheel_joint" type="fixed">
-    <parent link="base_link"/>
-    <child link="caster_wheel"/>
-    <origin xyz="${-base_l/4} 0.0 ${-base_h/2-wheel_r/2}" rpy="0.0 0.0 0.0"/>
-  </joint>
-  <joint name="imu_joint" type="fixed">
-    <parent link="base_link"/>
-    <child link="imu_link"/>
-    <origin xyz="${-base_l/4} 0.0 ${base_h/2+0.01}" rpy="0.0 0.0 0.0"/>
-  </joint>
-  <joint name="base_lidar_joint" type="fixed">
-    <parent link="base_link"/>
-    <child link="lidar_link"/>
-    <origin xyz="${base_l/4} 0.0 ${base_h/2+0.02}" rpy="0.0 0.0 0.0"/>
-  </joint>
+  <xacro:include filename="$(find marrtino_gazebo)/urdf/marrtino_base.urdf.xacro" />
+  <xacro:marrtino_base />
+  <xacro:marrtino_sensors />
+  <gazebo>
+    <!-- Joint state publisher -->
+    <plugin filename="gz_ros2_control-system" name="gz_ros2_control::GazeboSimROS2ControlPlugin">
+      <ros>
+        <namespace>$(arg namespace)</namespace>
+      </ros>
+      <parameters>$(find gz_ros2_control_demos)/config/diff_drive_controller.yaml</parameters>
+    </plugin>
+  </gazebo>
   <ros2_control name="GazeboSimSystem" type="system">
     <hardware>
@@ -181,12 +35,3 @@
     </joint>
   </ros2_control>
-  <gazebo>
-    <!-- Joint state publisher -->
-    <plugin filename="gz_ros2_control-system" name="gz_ros2_control::GazeboSimROS2ControlPlugin">
-      <ros>
-        <namespace>$(arg namespace)</namespace>
-      </ros>
-      <parameters>$(find gz_ros2_control_demos)/config/diff_drive_controller.yaml</parameters>
-    </plugin>
-  </gazebo>
 </robot>

Commit message: testing camera

File: marrtino_gazebo/urdf/marrtino.urdf.xacro (robot description, xacro)
@@ -3,4 +3,10 @@
   <xacro:arg name="namespace" default="" />
   <xacro:include filename="$(find marrtino_gazebo)/urdf/marrtino_base.urdf.xacro" />
+  <xacro:property name="wheel_r" value="0.06" />
+  <xacro:property name="wheel_max_velocity" value="${1 / wheel_r}" /> <!-- 1/r rad/s -> 1 m/s -->
+  <xacro:property name="arm_lower_limit" value="${-5*pi/4}" />
+  <xacro:property name="arm_upper_limit" value="${pi/4}" />
+  <xacro:property name="arm_max_effort" value="100" />
+  <xacro:property name="arm_max_velocity" value="1.0" />
   <xacro:marrtino_base />
   <xacro:marrtino_sensors />
@@ -13,4 +19,52 @@
       <parameters>$(find gz_ros2_control_demos)/config/diff_drive_controller.yaml</parameters>
     </plugin>
+    <plugin filename="gz-sim-imu-system"
+      name="gz::sim::systems::Imu">
+    </plugin>
+      <plugin filename="ImageDisplay" name="Image Display">
+        <gz-gui>
+          <property key="state" type="string">docked</property>
+        </gz-gui>
+        <topic>camera/image</topic>
+      </plugin>
+  </gazebo>
+  <gazebo reference="imu_link">
+    <sensor name="imu" type="imu">
+      <always_on>1</always_on>
+      <update_rate>10</update_rate>
+      <visualize>true</visualize>
+      <topic>imu</topic>
+      <enable_metrics>true</enable_metrics>
+    </sensor>
+  </gazebo>
+  <gazebo reference="camera_link">
+    <sensor name="camera" type="camera">
+      <camera>
+        <horizontal_fov>1.3962634</horizontal_fov>
+        <image>
+          <width>640</width>
+          <height>480</height>
+          <format>R8G8B8</format>
+        </image>
+        <clip>
+          <near>0.1</near>
+          <far>15</far>
+        </clip>
+        <noise>
+          <type>gaussian</type>
+          <!-- Noise is sampled independently per pixel on each frame.
+               That pixel's noise value is added to each of its color
+               channels, which at that point lie in the range [0,1]. -->
+          <mean>0.0</mean>
+          <stddev>0.007</stddev>
+        </noise>
+        <optical_frame_id>camera_link</optical_frame_id>
+        <camera_info_topic>camera/camera_info</camera_info_topic>
+      </camera>
+      <always_on>1</always_on>
+      <update_rate>10</update_rate>
+      <visualize>true</visualize>
+      <topic>camera/image</topic>
+    </sensor>
   </gazebo>
   <ros2_control name="GazeboSimSystem" type="system">
@@ -20,6 +74,6 @@
     <joint name="left_wheel_joint">
       <command_interface name="velocity">
-        <param name="min">${-max_velocity}</param>
-        <param name="max">${max_velocity}</param>
+        <param name="min">${-wheel_max_velocity}</param>
+        <param name="max">${wheel_max_velocity}</param>
       </command_interface>
       <state_interface name="position"/>
@@ -28,6 +82,6 @@
     <joint name="right_wheel_joint">
       <command_interface name="velocity">
-        <param name="min">${-max_velocity}</param>
-        <param name="max">${max_velocity}</param>
+        <param name="min">${-wheel_max_velocity}</param>
+        <param name="max">${wheel_max_velocity}</param>
       </command_interface>
       <state_interface name="position"/>

File: marrtino_gazebo/urdf/marrtino_base.urdf.xacro (robot description, xacro)
@@ -142,4 +142,20 @@
         </visual>
       </link>
+      <link name="camera_link">
+        <!--visual>
+          <origin xyz="0 0 0.03" rpy="0 0 0" />
+          <geometry>
+            <box size="0.02 0.02 0.06"/>
+          </geometry>
+          <material name="black"/>
+        </visual>
+        <visual name="visual_camera_frame">
+          <origin xyz="0 0 ${0.06+0.045}" rpy="0 0.5 0" />
+          <geometry>
+            <box size="0.02 0.12 0.09"/>
+          </geometry>
+          <material name="black"/>
+        </visual -->
+      </link>
       <link name="lidar_link">
         <visual>
@@ -155,4 +171,9 @@
         <child link="imu_link"/>
         <origin xyz="${-base_l/4} 0.0 ${base_h/2+0.01}" rpy="0.0 0.0 0.0"/>
+      </joint>
+      <joint name="camera_joint" type="fixed">
+        <parent link="base_link"/>
+        <child link="camera_link"/>
+        <origin xyz="0 0.0 ${base_h/2}" rpy="0.0 0.5 0.0"/>
       </joint>
       <joint name="base_lidar_joint" type="fixed">

Commit message: sensors OK

File: marrtino_gazebo/urdf/marrtino.urdf.xacro (robot description, xacro)
@@ -22,10 +22,10 @@
       name="gz::sim::systems::Imu">
     </plugin>
-      <plugin filename="ImageDisplay" name="Image Display">
+      <!-- plugin filename="ImageDisplay" name="Image Display">
         <gz-gui>
           <property key="state" type="string">docked</property>
         </gz-gui>
         <topic>camera/image</topic>
-      </plugin>
+      </plugin -->
   </gazebo>
   <gazebo reference="imu_link">
@@ -38,8 +38,39 @@
     </sensor>
   </gazebo>
-  <gazebo reference="camera_link">
+  <gazebo reference="lidar_link">
+    <sensor name="lidar" type="gpu_lidar">
+      <pose relative_to='lidar_link'>0 0 0.05 0 0 0</pose>
+      <always_on>1</always_on>
+      <update_rate>10</update_rate>
+      <visualize>true</visualize>
+      <topic>scan</topic>
+      <gz_frame_id>lidar_link</gz_frame_id>  <!-- ignore warning not defined in SDF -->
+      <ray>
+        <scan>
+            <horizontal>
+                <samples>640</samples>
+                <resolution>1</resolution>
+                <min_angle>${-pi*5/4}</min_angle>
+                <max_angle>${pi*5/4}</max_angle>
+            </horizontal>
+            <vertical>
+                <samples>1</samples>
+                <resolution>0.01</resolution>
+                <min_angle>0</min_angle>
+                <max_angle>0</max_angle>
+            </vertical>
+        </scan>
+        <range>
+            <min>0.05</min>
+            <max>10.0</max>
+            <resolution>0.01</resolution>
+        </range>
+      </ray>
+    </sensor>
+  </gazebo>
+  <gazebo reference="camera_optical_link">
     <sensor name="camera" type="camera">
       <camera>
-        <horizontal_fov>1.3962634</horizontal_fov>
+        <horizontal_fov>2.0</horizontal_fov>
         <image>
           <width>640</width>
@@ -48,5 +79,5 @@
         </image>
         <clip>
-          <near>0.1</near>
+          <near>0.001</near>
           <far>15</far>
         </clip>
@@ -59,5 +90,4 @@
           <stddev>0.007</stddev>
         </noise>
-        <optical_frame_id>camera_link</optical_frame_id>
         <camera_info_topic>camera/camera_info</camera_info_topic>
       </camera>

File: marrtino_gazebo/urdf/marrtino_2_arms.urdf.xacro (robot description, xacro)
@@ -20,4 +20,76 @@
       <parameters>$(find gz_ros2_control_demos)/config/diff_drive_controller.yaml</parameters>
     </plugin>
+    <plugin filename="gz-sim-imu-system"
+      name="gz::sim::systems::Imu">
+    </plugin>
+  </gazebo>
+  <gazebo reference="imu_link">
+    <sensor name="imu" type="imu">
+      <always_on>1</always_on>
+      <update_rate>10</update_rate>
+      <visualize>true</visualize>
+      <topic>imu</topic>
+      <enable_metrics>true</enable_metrics>
+    </sensor>
+  </gazebo>
+  <gazebo reference="lidar_link">
+    <sensor name="lidar" type="gpu_lidar">
+      <pose relative_to='lidar_link'>0 0 0.05 0 0 0</pose>
+      <always_on>1</always_on>
+      <update_rate>10</update_rate>
+      <visualize>true</visualize>
+      <topic>scan</topic>
+      <gz_frame_id>lidar_link</gz_frame_id>  <!-- ignore warning not defined in SDF -->
+      <ray>
+        <scan>
+            <horizontal>
+                <samples>640</samples>
+                <resolution>1</resolution>
+                <min_angle>${-pi*5/8}</min_angle>
+                <max_angle>${pi*5/8}</max_angle>
+            </horizontal>
+            <vertical>
+                <samples>1</samples>
+                <resolution>0.01</resolution>
+                <min_angle>0</min_angle>
+                <max_angle>0</max_angle>
+            </vertical>
+        </scan>
+        <range>
+            <min>0.05</min>
+            <max>10.0</max>
+            <resolution>0.01</resolution>
+        </range>
+      </ray>
+    </sensor>
+  </gazebo>
+  <gazebo reference="camera_optical_link">
+    <sensor name="camera" type="camera">
+      <camera>
+        <horizontal_fov>2.0</horizontal_fov>
+        <image>
+          <width>640</width>
+          <height>480</height>
+          <format>R8G8B8</format>
+        </image>
+        <clip>
+          <near>0.001</near>
+          <far>15</far>
+        </clip>
+        <noise>
+          <type>gaussian</type>
+          <!-- Noise is sampled independently per pixel on each frame.
+               That pixel's noise value is added to each of its color
+               channels, which at that point lie in the range [0,1]. -->
+          <mean>0.0</mean>
+          <stddev>0.007</stddev>
+        </noise>
+        <camera_info_topic>camera/camera_info</camera_info_topic>
+      </camera>
+      <always_on>1</always_on>
+      <update_rate>10</update_rate>
+      <visualize>true</visualize>
+      <topic>camera/image</topic>
+    </sensor>
   </gazebo>
   <ros2_control name="GazeboSimSystem" type="system">

File: marrtino_gazebo/urdf/marrtino_base.urdf.xacro (robot description, xacro)
@@ -18,5 +18,5 @@
       <xacro:property name="wheel_damping" value="0.05" />
       <xacro:property name="wheel_max_effort" value="100.0" />
-      <link name="base_footprint"/>
+      <link name="base_footprint" />
       <link name="base_link">
         <visual>
@@ -106,7 +106,7 @@
       </joint>
       <joint name="battery_joint" type="fixed">
-        <parent link="base_footprint"/>
+        <parent link="base_link"/>
         <child link="battery_link"/>
-        <origin xyz="${base_l/4} 0.0 ${wheel_r*2}" rpy="0.0 0.0 0.0"/>
+        <origin xyz="${base_l/4} 0.0 ${-wheel_r*2}" rpy="0.0 0.0 0.0"/>
       </joint>
       <joint name="left_wheel_joint" type="continuous">
@@ -142,19 +142,20 @@
         </visual>
       </link>
+      <link name="camera_optical_link" />
       <link name="camera_link">
-        <!--visual>
-          <origin xyz="0 0 0.03" rpy="0 0 0" />
+        <visual>
+          <origin xyz="0 0 0.05" rpy="0 0 0" />
           <geometry>
-            <box size="0.02 0.02 0.06"/>
+            <cylinder radius="0.01" length="0.10"/>
           </geometry>
           <material name="black"/>
         </visual>
-        <visual name="visual_camera_frame">
-          <origin xyz="0 0 ${0.06+0.045}" rpy="0 0.5 0" />
+        <visual>
+          <origin xyz="0.01 0 ${0.10+0.02}" rpy="0 ${pi/2+0.6} 0" />
           <geometry>
-            <box size="0.02 0.12 0.09"/>
+            <cylinder radius="0.02" length="0.02"/>
           </geometry>
           <material name="black"/>
-        </visual -->
+        </visual>
       </link>
       <link name="lidar_link">
@@ -175,5 +176,10 @@
         <parent link="base_link"/>
         <child link="camera_link"/>
-        <origin xyz="0 0.0 ${base_h/2}" rpy="0.0 0.5 0.0"/>
+        <origin xyz="0 0.0 ${base_h/2}" rpy="0.0 0.0 0.0"/>
+      </joint>
+      <joint name="camera_optical_joint" type="fixed">
+        <parent link="camera_link"/>
+        <child link="camera_optical_link"/>
+        <origin xyz="0.02 0 ${0.10+0.02}" rpy="0 0.6 0"/>
       </joint>
       <joint name="base_lidar_joint" type="fixed">
