Commit message: gtpose + many updates

File: marrtino_gazebo/urdf/marrtino.urdf.xacro (robot description, xacro)
@@ -2,4 +2,5 @@
 <robot name="marrtino" xmlns:xacro="http://ros.org/wiki/xacro">
   <xacro:arg name="namespace" default="" />
+  <xacro:arg name="battery_x_factor" default="1.0" />
   <xacro:include filename="$(find marrtino_gazebo)/urdf/marrtino_base.urdf.xacro" />
   <xacro:property name="wheel_r" value="0.06" />
@@ -9,5 +10,5 @@
   <xacro:property name="arm_max_effort" value="100" />
   <xacro:property name="arm_max_velocity" value="1.0" />
-  <xacro:marrtino_base />
+  <xacro:marrtino_base battery_x_factor="$(arg battery_x_factor)" />
   <xacro:marrtino_sensors />
   <gazebo>
@@ -21,4 +22,11 @@
     <plugin filename="gz-sim-imu-system"
       name="gz::sim::systems::Imu">
+    </plugin>
+    <plugin
+        filename="gz-sim-pose-publisher-system"
+        name="gz::sim::systems::PosePublisher">
+        <use_pose_vector_msg>false</use_pose_vector_msg>
+        <publish_model_pose>true</publish_model_pose>
+        <publish_nested_model_pose>true</publish_nested_model_pose>
     </plugin>
       <!-- plugin filename="ImageDisplay" name="Image Display">

File: marrtino_gazebo/urdf/marrtino_2_arms.urdf.xacro (robot description, xacro)
@@ -2,4 +2,5 @@
 <robot name="ddrive_robot" xmlns:xacro="http://ros.org/wiki/xacro">
   <xacro:arg name="namespace" default="" />
+  <xacro:arg name="battery_x_factor" default="1.0" />
   <xacro:include filename="$(find marrtino_gazebo)/urdf/marrtino_base.urdf.xacro" />
   <xacro:property name="wheel_r" value="0.06" />
@@ -9,5 +10,5 @@
   <xacro:property name="arm_max_effort" value="100" />
   <xacro:property name="arm_max_velocity" value="1.0" />
-  <xacro:marrtino_base />
+  <xacro:marrtino_base battery_x_factor="$(arg battery_x_factor)" />
   <xacro:marrtino_sensors />
   <xacro:marrtino_arms />
@@ -22,4 +23,11 @@
     <plugin filename="gz-sim-imu-system"
       name="gz::sim::systems::Imu">
+    </plugin>
+    <plugin
+        filename="gz-sim-pose-publisher-system"
+        name="gz::sim::systems::PosePublisher">
+        <use_pose_vector_msg>false</use_pose_vector_msg>
+        <publish_model_pose>true</publish_model_pose>
+        <publish_nested_model_pose>true</publish_nested_model_pose>
     </plugin>
   </gazebo>

File: marrtino_gazebo/urdf/marrtino_base.urdf.xacro (robot description, xacro)
@@ -13,9 +13,10 @@
   <xacro:property name="base_l" value="0.30" />
   <xacro:property name="base_h" value="0.20" />
-  <xacro:macro name="marrtino_base">
+  <xacro:macro name="marrtino_base" params="battery_x_factor">
       <xacro:property name="wheel_l" value="0.03" />
       <xacro:property name="wheel_friction" value="0.01" />
       <xacro:property name="wheel_damping" value="0.05" />
       <xacro:property name="wheel_max_effort" value="100.0" />
+      <xacro:property name="battery_x" value="${battery_x_factor*base_l/4}" />
       <link name="base_footprint" />
       <link name="base_link">
@@ -103,10 +104,10 @@
         <parent link="base_footprint"/>
         <child link="base_link"/>
-        <origin xyz="0.0 0.0 ${base_h/2+wheel_r}" rpy="0.0 0.0 0.0"/>
+        <origin xyz="${-base_l/4} 0.0 ${base_h/2+wheel_r}" rpy="0.0 0.0 0.0"/>
       </joint>
       <joint name="battery_joint" type="fixed">
         <parent link="base_link"/>
         <child link="battery_link"/>
-        <origin xyz="${base_l/4} 0.0 ${-wheel_r*2}" rpy="0.0 0.0 0.0"/>
+        <origin xyz="${battery_x} 0.0 ${-wheel_r*2}" rpy="0.0 0.0 0.0"/>
       </joint>
       <joint name="left_wheel_joint" type="continuous">

File: marrtino_gazebo/urdf/smarrtino.urdf.xacro (robot description, xacro)
@@ -384,4 +384,11 @@
     <plugin filename="gz-sim-imu-system"
       name="gz::sim::systems::Imu">
+    </plugin>
+    <plugin
+        filename="gz-sim-pose-publisher-system"
+        name="gz::sim::systems::PosePublisher">
+        <use_pose_vector_msg>false</use_pose_vector_msg>
+        <publish_model_pose>true</publish_model_pose>
+        <publish_nested_model_pose>true</publish_nested_model_pose>
     </plugin>
   </gazebo>
