Commit message: smarrtino control OK

File: marrtino_gazebo/urdf/smarrtino.urdf.xacro (robot description, xacro)
@@ -2,7 +2,5 @@
 <robot name="smarrtino" xmlns:xacro="http://ros.org/wiki/xacro">
   <xacro:arg name="namespace" default="" />
-  <xacro:property name="head_mass" value="0.10" />
-  <xacro:property name="body_mass" value="0.40" />
-  <xacro:property name="head_radius" value="0.05" />
+  <xacro:property name="body_mass" value="0.60" />
   <xacro:property name="body_radius" value="0.1" />
   <xacro:property name="base_w" value="0.22" />
@@ -11,6 +9,6 @@
   <xacro:property name="wheel_r" value="0.05" />
   <xacro:property name="wheel_l" value="0.02" />
-  <xacro:property name="friction" value="0.02" />
-  <xacro:property name="damping" value="0.09" />
+  <xacro:property name="friction" value="0.001" />
+  <xacro:property name="damping" value="0.001" />
   <xacro:property name="max_effort" value="1000.0" />
   <xacro:property name="max_velocity" value="100.0" />
@@ -20,6 +18,12 @@
   <xacro:property name="arm_max_effort" value="30.0" />
   <xacro:property name="arm_max_velocity" value="1.0" />
-  <xacro:property name="arm_friction" value="0.01" />
+  <xacro:property name="arm_friction" value="0.001" />
   <xacro:property name="arm_damping" value="0.01" />
+  <xacro:property name="head_mass" value="0.10" />
+  <xacro:property name="head_radius" value="0.05" />
+  <xacro:property name="head_max_effort" value="30.0" />
+  <xacro:property name="head_max_velocity" value="1.0" />
+  <xacro:property name="head_friction" value="0.02" />
+  <xacro:property name="head_damping" value="0.02" />
   <xacro:include filename="$(find marrtino_gazebo)/urdf/inertia.xacro" />
   <material name="orange"><color rgba="1.0 0.33 0.0 1.0"/></material>
@@ -106,4 +110,5 @@
     <xacro:sphere_inertial mass="0.2" radius="${wheel_r/2}" />
   </link>
+  <link name="top_base_link" />
   <link name="head_link">
     <visual>
@@ -112,5 +117,12 @@
       </geometry>
       <origin xyz="0.02 0 -0.4" rpy="0 0 ${pi/2}"/>
-      <material name="white"/>
+      <material name="orange"/>
+    </visual>
+    <visual>
+      <geometry>
+          <cylinder radius="0.06" length="0.002"/>
+      </geometry>
+      <origin xyz="0.045 0 0.01" rpy="0 ${pi/2} 0"/>
+      <material name="black"/>
     </visual>
     <collision>
@@ -122,5 +134,5 @@
     <xacro:sphere_inertial_roll mass="${head_mass}" radius="${head_radius}" roll="${pi/2}"/>
   </link>
-  <link name="head_base_link">
+  <link name="base_head_link">
     <visual>
         <geometry>
@@ -130,4 +142,14 @@
         <material name="blue"/>
     </visual>
+  </link>
+  <link name="tilt_head_link">
+    <visual>
+        <geometry>
+            <cylinder radius="0.02" length="0.04"/>
+        </geometry>
+        <origin xyz="0.0 0.0 0.0" rpy="0.0 ${pi/2} ${pi/2}"/>
+        <material name="green"/>
+    </visual>
+    <xacro:sphere_inertial mass="0.01" radius="0.01" />
   </link>
   <link name="imu_link">
@@ -154,15 +176,29 @@
     <origin xyz="0 0 0.02" rpy="0 0.0 0.0"/>
   </joint>
-  <joint name="head_pan_joint" type="revolute">
+  <joint name="top_base_joint" type="fixed">
     <parent link="base_link"/>
-    <child link="head_base_link"/>
-    <origin xyz="-0.06 0 ${base_h}" rpy="0 0 0"/>
+    <child link="top_base_link"/>
+    <origin xyz="-0.06 0 ${base_h}" rpy="0 0.0 0.0"/>
+  </joint>
+  <joint name="tilt_head_joint" type="revolute">
+    <parent link="top_base_link"/>
+    <child link="tilt_head_link"/>
+    <origin xyz="0 0 0.01" rpy="0 0 0"/>
+    <axis xyz="0 1 0"/>
+    <dynamics damping="${head_damping}" friction="${head_friction}"/>
+    <limit effort="${head_max_effort}" velocity="${head_max_velocity}"
+           lower="${-pi/4}" upper="${pi/4}" />
+  </joint>
+  <joint name="pan_head_joint" type="revolute">
+    <parent link="tilt_head_link"/>
+    <child link="base_head_link"/>
+    <origin xyz="0 0 0.01" rpy="0 0 0"/>
     <axis xyz="0 0 1"/>
-    <dynamics damping="${arm_damping}" friction="${arm_friction}"/>
-    <limit effort="${arm_max_effort}" velocity="${arm_max_velocity}"
+    <dynamics damping="${head_damping}" friction="${head_friction}"/>
+    <limit effort="${head_max_effort}" velocity="${head_max_velocity}"
            lower="${-pi/2}" upper="${pi/2}" />
   </joint>
-  <joint name="head_base_joint" type="fixed">
-    <parent link="head_base_link"/>
+  <joint name="base_head_joint" type="fixed">
+    <parent link="base_head_link"/>
     <child link="head_link"/>
     <origin xyz="0 0 0.07" rpy="0 0 0"/>
@@ -197,5 +233,5 @@
     <parent link="base_link"/>
     <child link="lidar_link"/>
-    <origin xyz="-0.02 0 0.05" rpy="0.0 0.0 0.0"/>
+    <origin xyz="0.04 0 0.06" rpy="0.0 0.0 0.0"/>
   </joint>
   <link name="left_arm_body">
@@ -235,5 +271,5 @@
         </geometry>
         <origin xyz="0.065 -0.09 -0.265" rpy="0 0 ${pi/2}"/>
-        <material name="white"/>
+        <material name="green"/>
     </visual>
     <collision>
@@ -262,5 +298,5 @@
         </geometry>
         <origin xyz="0.065 0.09 -0.265" rpy="0 0 ${pi/2}"/>
-        <material name="white"/>
+        <material name="green"/>
     </visual>
     <collision>
@@ -317,6 +353,6 @@
     <joint name="left_wheel_joint">
       <command_interface name="velocity">
-        <param name="min">-10</param>
-        <param name="max">10</param>
+        <param name="min">${-max_velocity}</param>
+        <param name="max">${max_velocity}</param>
       </command_interface>
       <state_interface name="position"/>
@@ -325,6 +361,6 @@
     <joint name="right_wheel_joint">
       <command_interface name="velocity">
-        <param name="min">-10</param>
-        <param name="max">10</param>
+        <param name="min">${-max_velocity}</param>
+        <param name="max">${max_velocity}</param>
       </command_interface>
       <state_interface name="position"/>
@@ -340,4 +376,20 @@
     </joint>
     <joint name="right_arm_joint">
+      <command_interface name="effort">
+        <param name="min">-10</param>
+        <param name="max">10</param>
+      </command_interface>
+      <state_interface name="position"/>
+      <state_interface name="velocity"/>
+    </joint>
+    <joint name="pan_head_joint">
+      <command_interface name="effort">
+        <param name="min">-10</param>
+        <param name="max">10</param>
+      </command_interface>
+      <state_interface name="position"/>
+      <state_interface name="velocity"/>
+    </joint>
+    <joint name="tilt_head_joint">
       <command_interface name="effort">
         <param name="min">-10</param>

Commit message: smarrtino face

File: marrtino_gazebo/urdf/smarrtino.urdf.xacro (robot description, xacro)
@@ -34,4 +34,5 @@
   <material name="grey"><color rgba="0.7 0.7 0.7 1.0"/></material>
   <material name="white"><color rgba="1 1 1 1.0"/></material>
+  <material name="green_t"><color rgba="0 1 0 0.5"/></material>
   <link name="base_footprint"/>
   <link name="base_link">
@@ -126,4 +127,17 @@
       <material name="black"/>
     </visual>
+    <visual>
+      <geometry>
+          <cylinder radius="0.06" length="0.002"/>
+      </geometry>
+      <origin xyz="0.045 0 0.01" rpy="0 ${pi/2} 0"/>
+      <material name="black"/>
+    </visual>
+    <visual name="front">
+      <origin xyz="0.047 0 -0.04" rpy="0 0 0"/>
+      <geometry>
+        <mesh filename="$(find marrtino_gazebo)/urdf/meshes/face.dae" scale="0.01 0.20 0.20" />
+      </geometry>
+    </visual>
     <collision>
       <geometry>

Commit message: smarrtino sensors

File: marrtino_gazebo/urdf/smarrtino.urdf.xacro (robot description, xacro)
@@ -173,4 +173,13 @@
     <xacro:sphere_inertial mass="0.01" radius="0.01" />
   </link>
+  <link name="camera_optical_link">
+    <visual>
+        <geometry>
+            <cylinder radius="0.005" length="0.005"/>
+        </geometry>
+        <origin xyz="0.0 0.0 0.0" rpy="0.0 ${pi/2} 0.0"/>
+        <material name="white"/>
+    </visual>
+  </link>
   <link name="imu_link">
     <visual>
@@ -223,4 +232,9 @@
     <child link="head_link"/>
     <origin xyz="0 0 0.07" rpy="0 0 0"/>
+  </joint>
+  <joint name="camera_optical_joint" type="fixed">
+    <parent link="head_link"/>
+    <child link="camera_optical_link"/>
+    <origin xyz="0.048 0 0.07" rpy="0 0 0"/>
   </joint>
   <joint name="left_wheel_joint" type="continuous">
@@ -367,4 +381,78 @@
     <origin xyz="0 -0.02 0" rpy="0 0.0 0.0"/>
   </joint>
+  <gazebo>
+    <plugin filename="gz-sim-imu-system"
+      name="gz::sim::systems::Imu">
+    </plugin>
+  </gazebo>
+  <gazebo reference="imu_link">
+    <sensor name="imu" type="imu">
+      <always_on>1</always_on>
+      <update_rate>10</update_rate>
+      <visualize>true</visualize>
+      <topic>imu</topic>
+      <enable_metrics>true</enable_metrics>
+    </sensor>
+  </gazebo>
+  <gazebo reference="lidar_link">
+    <sensor name="lidar" type="gpu_lidar">
+      <pose relative_to='lidar_link'>0.021 0 0 0 0 0</pose>
+      <always_on>1</always_on>
+      <update_rate>10</update_rate>
+      <visualize>true</visualize>
+      <topic>scan</topic>
+      <gz_frame_id>lidar_link</gz_frame_id>  <!-- ignore warning not defined in SDF -->
+      <ray>
+        <scan>
+            <horizontal>
+                <samples>640</samples>
+                <resolution>1</resolution>
+                <min_angle>${-pi*3/8}</min_angle>
+                <max_angle>${pi*3/8}</max_angle>
+            </horizontal>
+            <vertical>
+                <samples>1</samples>
+                <resolution>0.01</resolution>
+                <min_angle>0</min_angle>
+                <max_angle>0</max_angle>
+            </vertical>
+        </scan>
+        <range>
+            <min>0.05</min>
+            <max>10.0</max>
+            <resolution>0.01</resolution>
+        </range>
+      </ray>
+    </sensor>
+  </gazebo>
+  <gazebo reference="camera_optical_link">
+    <sensor name="camera" type="camera">
+      <camera>
+        <horizontal_fov>2.0</horizontal_fov>
+        <image>
+          <width>640</width>
+          <height>480</height>
+          <format>R8G8B8</format>
+        </image>
+        <clip>
+          <near>0.001</near>
+          <far>15</far>
+        </clip>
+        <noise>
+          <type>gaussian</type>
+          <!-- Noise is sampled independently per pixel on each frame.
+               That pixel's noise value is added to each of its color
+               channels, which at that point lie in the range [0,1]. -->
+          <mean>0.0</mean>
+          <stddev>0.007</stddev>
+        </noise>
+        <camera_info_topic>camera/camera_info</camera_info_topic>
+      </camera>
+      <always_on>1</always_on>
+      <update_rate>10</update_rate>
+      <visualize>true</visualize>
+      <topic>camera/image</topic>
+    </sensor>
+  </gazebo>
   <ros2_control name="GazeboSimSystem" type="system">
     <hardware>

Commit message: top camera

File: marrtino_gazebo/urdf/smarrtino.urdf.xacro (robot description, xacro)
@@ -495,4 +495,47 @@
     </sensor>
   </gazebo>
+  <!-- top view camera -->
+  <link name="top_camera_link">
+    <visual>
+      <geometry>
+        <cylinder radius="0.005" length="0.006"/>
+      </geometry>
+      <material name="grey"/>
+      <origin xyz="0 0 0" rpy="0 0 0" />
+    </visual>
+  </link>
+  <link name="top_camera_optical_link" />
+  <joint name="top_camera_joint" type="fixed">
+    <parent link="base_footprint"/>
+    <child link="top_camera_link"/>
+    <origin xyz="0 0 2" rpy="0.0 ${pi} 0.0"/>
+  </joint>
+  <joint name="top_camera_optical_joint" type="fixed">
+    <parent link="top_camera_link"/>
+    <child link="top_camera_optical_link"/>
+    <origin xyz="0 0 0.006" rpy="0 ${-pi/2} 0"/>
+  </joint>
+  <gazebo reference="top_camera_optical_link">
+    <sensor name="top_camera" type="camera">
+      <camera>
+        <horizontal_fov>2.0</horizontal_fov>
+        <image>
+          <width>640</width>
+          <height>480</height>
+          <format>R8G8B8</format>
+        </image>
+        <clip>
+          <near>0.001</near>
+          <far>15</far>
+        </clip>
+        <camera_info_topic>top_camera/camera_info</camera_info_topic>
+      </camera>
+      <always_on>1</always_on>
+      <update_rate>10</update_rate>
+      <visualize>true</visualize>
+      <topic>top_camera/image</topic>
+      <gz_frame_id>top_camera_optical_link</gz_frame_id>  <!-- ignore warning not defined in SDF -->
+    </sensor>
+  </gazebo>
   <ros2_control name="GazeboSimSystem" type="system">
     <hardware>

Commit message: cpu reduce

File: marrtino_gazebo/urdf/smarrtino.urdf.xacro (robot description, xacro)
@@ -52,8 +52,14 @@
     <collision>
       <geometry>
+        <box size="${base_l+0.03} ${base_w+0.10} ${base_h}"/>
+      </geometry>
+      <origin xyz="-0.05 0 ${base_h/2}" rpy="0 0 0"/>
+    </collision>
+    <!-- collision>
+      <geometry>
         <mesh filename="$(find marrtino_gazebo)/urdf/meshes/smarrtino_body.stl" scale="0.001 0.001 0.001"/>
       </geometry>
       <origin xyz="0 0 0" rpy="0 0 ${pi/2}"/>
-    </collision>
+    </collision -->
     <inertial>
       <origin xyz="0 0 0.1" rpy="0 0 0"/>
@@ -181,8 +187,14 @@
     <collision>
       <geometry>
+        <sphere radius="${head_radius+0.05}"/>
+      </geometry>
+      <origin xyz="-0.02 0 0.02" rpy="0 0 ${pi/2}"/>
+    </collision>
+    <!-- collision>
+      <geometry>
         <mesh filename="$(find marrtino_gazebo)/urdf/meshes/smarrtino_head.stl" scale="0.001 0.001 0.001"/>
       </geometry>
       <origin xyz="0.02 0 -0.4" rpy="0 0 ${pi/2}"/>
-    </collision>
+    </collision -->
     <xacro:sphere_inertial_roll mass="${head_mass}" radius="${head_radius}" roll="${pi/2}"/>
   </link>
@@ -340,10 +352,10 @@
         <material name="green"/>
     </visual>
-    <collision>
+    <!-- collision>
         <geometry>
           <mesh filename="$(find marrtino_gazebo)/urdf/meshes/smarrtino_arm_left.stl" scale="0.001 0.001 0.001"/>
         </geometry>
         <origin xyz="0.065 -0.09 -0.265" rpy="0 0 ${pi/2}"/>
-    </collision>
+    </collision -->
     <inertial>
       <origin xyz="0 0.045 -0.07" rpy="0.3 0 0"/>
@@ -367,10 +379,10 @@
         <material name="green"/>
     </visual>
-    <collision>
+    <!-- collision>
         <geometry>
           <mesh filename="$(find marrtino_gazebo)/urdf/meshes/smarrtino_arm_right.stl" scale="0.001 0.001 0.001"/>
         </geometry>
         <origin xyz="0.065 0.09 -0.265" rpy="0 0 ${pi/2}"/>
-    </collision>
+    </collision -->
     <inertial>
       <origin xyz="0 -0.045 -0.07" rpy="-0.3 0 0"/>
@@ -496,4 +508,6 @@
   </gazebo>
   <!-- top view camera -->
+  <xacro:arg name="topview_camera" default="false" />
+  <xacro:if value="$(arg topview_camera)">
   <link name="top_camera_link">
     <visual>
@@ -521,6 +535,6 @@
         <horizontal_fov>2.0</horizontal_fov>
         <image>
-          <width>640</width>
-          <height>480</height>
+          <width>320</width>
+          <height>240</height>
           <format>R8G8B8</format>
         </image>
@@ -532,5 +546,5 @@
       </camera>
       <always_on>1</always_on>
-      <update_rate>10</update_rate>
+      <update_rate>1</update_rate>
       <visualize>true</visualize>
       <topic>top_camera/image</topic>
@@ -538,4 +552,5 @@
     </sensor>
   </gazebo>
+  </xacro:if>
   <ros2_control name="GazeboSimSystem" type="system">
     <hardware>
